File: KiCad Project Files/esp32 pcb.kicad_sch (KiCad schematic)
At the start: 28 parts, among them U1 ESP32-S3-MINI-1-N8, U2 D3V3XA4B10LP, U3 TLV75801PDRV, U4 ENS210

Commit message: Don't know if it worked but tried to make the project self contained - can fix later if it didn't work
Parts:
- renumbered BOOT to BOOT1, JUSB to JUSB1, RESET to RESET1
Changed lines of the file:
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@@
 		(dnp no)
 		(fields_autoplaced yes)
-		(property "Reference" "RESET"
+		(property "Reference" "RESET1"
 			(at 113.03 63.5 0)
 			(show_name no)
@@
 			(project "esp32 pcb"
 				(path "/afce35cb-236d-4e62-a028-55190f12758c"
-					(reference "RESET")
+					(reference "RESET1")
 					(unit 1)
 				)
@@
 		(dnp no)
 		(fields_autoplaced yes)
-		(property "Reference" "BOOT"
+		(property "Reference" "BOOT1"
 			(at 113.03 83.82 0)
 			(show_name no)
@@
 			(project "esp32 pcb"
 				(path "/afce35cb-236d-4e62-a028-55190f12758c"
-					(reference "BOOT")
+					(reference "BOOT1")
 					(unit 1)
 				)
@@
 		(dnp no)
 		(fields_autoplaced yes)
-		(property "Reference" "JUSB"
+		(property "Reference" "JUSB1"
 			(at 35.56 57.15 0)
 			(show_name no)
@@
 			(project "esp32 pcb"
 				(path "/afce35cb-236d-4e62-a028-55190f12758c"
-					(reference "JUSB")
-					(unit 1)
-				)
+					(reference "JUSB1")
+					(unit 1)
+				)
